File: air_test1/air_test1.kicad_pcb (KiCad board)
At the start: 2 copper layers, 82.5 x 58 mm, 21 parts, among them J1 Conn_01x02_Pin, J2 Conn_01x02_Pin, J3 Conn_01x02_Pin, J4 Conn_01x02_Pin, J5 Conn_01x02_Pin, J6 Conn_01x04_Pin, J7 Conn_01x03_Pin, J8 Conn_01x03_Pin

Commit message: update some data and add garber
Parts:
- added G***: LOGO, marc, B.Cu at (137.5, 108.0)
Other:
- board text added: "1 2 3 4"
- board text added: "2024,10"
- board text added: "Max Current 1.5A/4ch"
- board text added: "Solenoid Valve Controller V1.0"
- board text added: "①"
- board text added: "②"
- board text added: "③"
- board text added: "④"
- board text removed: "Max Current 1.5A/ch"
- board text removed: "Solenoid Vavle Controller V1.0"

Commit message: upload new project
Parts:
- removed G***: LOGO, marc
